File: quadcopter.sch (EAGLE design)
At the start: 66 parts, among them J1 AVR_SPI_PRG_6NS, Q1 2.6A, Q2 2.6A, Q3 2.6A, Q4 2.6A, U1 ATMEGA128RFA1, U2 IMU_LSM9DS1TR, Y1 16MHz

Commit message: Some changes based on design reviews
Parts:
- removed C9: 1uF, quadparts_prebuilt:CAPACITOR-NP_SMD-2012-0805_CERAMIC-1UF
- added C17: 0.1uF, quadparts_prebuilt:CAPACITOR-NP_SMD-2012-0805_CERAMIC-0.1UF
- C3, C5, C7: value 1uF -> 0.1uF; device quadparts_prebuilt:CAPACITOR-NP_SMD-2012-0805_CERAMIC-1UF -> quadparts_prebuilt:CAPACITOR-NP_SMD-2012-0805_CERAMIC-0.1UF
Connections:
- net BAT_GND: now also C10.2, C17.2; no longer C9.2
- net FILTERED: now also C7.1; no longer C9.1
- net GND: no longer C10.2
- net N$31: now also C3.1; no longer C7.1
- net N$33: now also C17.1; no longer C3.1
- net RX0: now also U1.PE1(TXD0); no longer U1.PE0(RXD0/PCINT8)
- net TX0: now also U1.PE0(RXD0/PCINT8); no longer U1.PE1(TXD0)
Other:
- moved on the sheet: C3, C7
Changed lines of the file:
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@@
 <part name="C8" library="quadparts_prebuilt" deviceset="CAPACITOR-POL_" device="SMD-7043-D_TANTALUM-220UF" value="220uF"/>
 <part name="Q4" library="quadparts_connie" deviceset="N_MOSFET_SI2302CDS_T1_E3" device="" value="2.6A"/>
-<part name="C9" library="quadparts_prebuilt" deviceset="CAPACITOR-NP_" device="SMD-2012-0805_CERAMIC-1UF" value="1uF"/>
 <part name="D4" library="quadparts_prebuilt" deviceset="DIODE-SCHOTTKY_" device="SMD-SOD123"/>
 <part name="U$2" library="quadparts_prebuilt" deviceset="MOTOR_PADS" device=""/>
 <part name="C2" library="quadparts_prebuilt" deviceset="CAPACITOR-POL_" device="SMD-7043-D_TANTALUM-220UF" value="220uF"/>
 <part name="Q1" library="quadparts_connie" deviceset="N_MOSFET_SI2302CDS_T1_E3" device="" value="2.6A"/>
-<part name="C3" library="quadparts_prebuilt" deviceset="CAPACITOR-NP_" device="SMD-2012-0805_CERAMIC-1UF" value="1uF"/>
 <part name="D1" library="quadparts_prebuilt" deviceset="DIODE-SCHOTTKY_" device="SMD-SOD123"/>
 <part name="U$4" library="quadparts_prebuilt" deviceset="MOTOR_PADS" device=""/>
 <part name="C4" library="quadparts_prebuilt" deviceset="CAPACITOR-POL_" device="SMD-7043-D_TANTALUM-220UF" value="220uF"/>
 <part name="Q2" library="quadparts_connie" deviceset="N_MOSFET_SI2302CDS_T1_E3" device="" value="2.6A"/>
-<part name="C5" library="quadparts_prebuilt" deviceset="CAPACITOR-NP_" device="SMD-2012-0805_CERAMIC-1UF" value="1uF"/>
 <part name="D2" library="quadparts_prebuilt" deviceset="DIODE-SCHOTTKY_" device="SMD-SOD123"/>
 <part name="U$5" library="quadparts_prebuilt" deviceset="MOTOR_PADS" device=""/>
 <part name="C6" library="quadparts_prebuilt" deviceset="CAPACITOR-POL_" device="SMD-7043-D_TANTALUM-220UF" value="220uF"/>
 <part name="Q3" library="quadparts_connie" deviceset="N_MOSFET_SI2302CDS_T1_E3" device="" value="2.6A"/>
-<part name="C7" library="quadparts_prebuilt" deviceset="CAPACITOR-NP_" device="SMD-2012-0805_CERAMIC-1UF" value="1uF"/>
 <part name="D3" library="quadparts_prebuilt" deviceset="DIODE-SCHOTTKY_" device="SMD-SOD123"/>
 <part name="C10" library="quadparts_prebuilt" deviceset="CAPACITOR-NP_" device="SMD-2012-0805_CERAMIC-1UF" value="1uF"/>
@@
 <part name="R10" library="quadparts_prebuilt" deviceset="RESISTOR_" device="SMD-2012-0805-100" value="100"/>
 <part name="R11" library="quadparts_prebuilt" deviceset="RESISTOR_" device="SMD-2012-0805-100" value="100"/>
+<part name="C17" library="quadparts_prebuilt" deviceset="CAPACITOR-NP_" device="SMD-2012-0805_CERAMIC-0.1UF" value="0.1uF"/>
+<part name="C3" library="quadparts_prebuilt" deviceset="CAPACITOR-NP_" device="SMD-2012-0805_CERAMIC-0.1UF" value="0.1uF"/>
+<part name="C5" library="quadparts_prebuilt" deviceset="CAPACITOR-NP_" device="SMD-2012-0805_CERAMIC-0.1UF" value="0.1uF"/>
+<part name="C7" library="quadparts_prebuilt" deviceset="CAPACITOR-NP_" device="SMD-2012-0805_CERAMIC-0.1UF" value="0.1uF"/>
 </parts>
 <sheets>
@@
 <instance part="C8" gate="G$1" x="-162.56" y="-48.26"/>
 <instance part="Q4" gate="G$1" x="-137.16" y="-88.9"/>
-<instance part="C9" gate="G$1" x="-162.56" y="-99.06"/>
 <instance part="D4" gate="G$1" x="-121.92" y="-48.26" rot="R90"/>
 <instance part="U$2" gate="G$1" x="-142.24" y="101.6"/>
 <instance part="C2" gate="G$1" x="-162.56" y="104.14"/>
 <instance part="Q1" gate="G$1" x="-137.16" y="63.5"/>
-<instance part="C3" gate="G$1" x="-162.56" y="53.34"/>
 <instance part="D1" gate="G$1" x="-121.92" y="104.14" rot="R90"/>
 <instance part="U$4" gate="G$1" x="144.78" y="-50.8"/>
 <instance part="C4" gate="G$1" x="124.46" y="-48.26"/>
 <instance part="Q2" gate="G$1" x="149.86" y="-88.9"/>
-<instance part="C5" gate="G$1" x="124.46" y="-99.06"/>
 <instance part="D2" gate="G$1" x="165.1" y="-48.26" rot="R90"/>
 <instance part="U$5" gate="G$1" x="99.06" y="101.6"/>
 <instance part="C6" gate="G$1" x="78.74" y="104.14"/>
 <instance part="Q3" gate="G$1" x="104.14" y="63.5"/>
-<instance part="C7" gate="G$1" x="78.74" y="53.34"/>
 <instance part="D3" gate="G$1" x="119.38" y="104.14" rot="R90"/>
 <instance part="C10" gate="G$1" x="-182.88" y="-2.54"/>
@@
 <instance part="R10" gate="G$1" x="-93.98" y="78.74" rot="R270"/>
 <instance part="R11" gate="G$1" x="-114.3" y="78.74" rot="R180"/>
+<instance part="C17" gate="G$1" x="-162.56" y="53.34"/>
+<instance part="C3" gate="G$1" x="78.74" y="53.34"/>
+<instance part="C5" gate="G$1" x="124.46" y="-99.06"/>
+<instance part="C7" gate="G$1" x="-162.56" y="-99.06"/>
 </instances>
 <busses>
@@
 <label x="-134.62" y="15.24" size="1.778" layer="95" rot="R180"/>
 <pinref part="GND7" gate="1" pin="GND"/>
-</segment>
-<segment>
-<pinref part="C10" gate="G$1" pin="2"/>
-<wire x1="-182.88" y1="-7.62" x2="-182.88" y2="-10.16" width="0.1524" layer="91"/>
-<label x="-185.42" y="-12.7" size="1.778" layer="95"/>
 </segment>
 <segment>
@@
 <net name="RX0" class="0">
 <segment>
-<pinref part="U1" gate="G$1" pin="PE0(RXD0/PCINT8)"/>
-<wire x1="-83.82" y1="-20.32" x2="-91.44" y2="-20.32" width="0.1524" layer="91"/>
-<label x="-53.34" y="73.66" size="1.778" layer="95"/>
-<label x="-91.44" y="-20.32" size="1.778" layer="95"/>
-</segment>
-</net>
-<net name="TX0" class="0">
-<segment>
 <pinref part="U1" gate="G$1" pin="PE1(TXD0)"/>
 <wire x1="-83.82" y1="-22.86" x2="-91.44" y2="-22.86" width="0.1524" layer="91"/>
@@
 <pinref part="R6" gate="G$1" pin="2"/>
 <wire x1="-162.56" y1="-91.44" x2="-162.56" y2="-96.52" width="0.1524" layer="91"/>
-<pinref part="C9" gate="G$1" pin="1"/>
 <wire x1="-152.4" y1="-91.44" x2="-162.56" y2="-91.44" width="0.1524" layer="91"/>
 <pinref part="R15" gate="G$1" pin="2"/>
 <junction x="-162.56" y="-91.44"/>
+<pinref part="C7" gate="G$1" pin="1"/>
 </segment>
 </net>
@@
 <wire x1="-172.72" y1="-111.76" x2="-162.56" y2="-111.76" width="0.1524" layer="91"/>
 <junction x="-152.4" y="-111.76"/>
-<pinref part="C9" gate="G$1" pin="2"/>
 <wire x1="-162.56" y1="-111.76" x2="-152.4" y2="-111.76" width="0.1524" layer="91"/>
 <wire x1="-162.56" y1="-104.14" x2="-162.56" y2="-111.76" width="0.1524" layer="91"/>
@@
 <label x="-175.26" y="-114.3" size="1.778" layer="95"/>
 <pinref part="R6" gate="G$1" pin="1"/>
+<pinref part="C7" gate="G$1" pin="2"/>
 </segment>
 <segment>
@@
 <wire x1="-172.72" y1="40.64" x2="-162.56" y2="40.64" width="0.1524" layer="91"/>
 <junction x="-152.4" y="40.64"/>
-<pinref part="C3" gate="G$1" pin="2"/>
 <wire x1="-162.56" y1="40.64" x2="-152.4" y2="40.64" width="0.1524" layer="91"/>
 <wire x1="-162.56" y1="48.26" x2="-162.56" y2="40.64" width="0.1524" layer="91"/>
@@
 <label x="-175.26" y="38.1" size="1.778" layer="95"/>
 <pinref part="R3" gate="G$1" pin="1"/>
+<pinref part="C17" gate="G$1" pin="2"/>
 </segment>
 <segment>
@@
 <wire x1="114.3" y1="-111.76" x2="124.46" y2="-111.76" width="0.1524" layer="91"/>
 <junction x="134.62" y="-111.76"/>
-<pinref part="C5" gate="G$1" pin="2"/>
 <wire x1="124.46" y1="-111.76" x2="134.62" y2="-111.76" width="0.1524" layer="91"/>
 <wire x1="124.46" y1="-104.14" x2="124.46" y2="-111.76" width="0.1524" layer="91"/>
@@
 <label x="111.76" y="-114.3" size="1.778" layer="95"/>
 <pinref part="R16" gate="G$1" pin="1"/>
+<pinref part="C5" gate="G$1" pin="2"/>
 </segment>
 <segment>
@@
 <wire x1="68.58" y1="40.64" x2="78.74" y2="40.64" width="0.1524" layer="91"/>
 <junction x="88.9" y="40.64"/>
-<pinref part="C7" gate="G$1" pin="2"/>
 <wire x1="78.74" y1="40.64" x2="88.9" y2="40.64" width="0.1524" layer="91"/>
 <wire x1="78.74" y1="48.26" x2="78.74" y2="40.64" width="0.1524" layer="91"/>
@@
 <label x="66.04" y="38.1" size="1.778" layer="95"/>
 <pinref part="R4" gate="G$1" pin="1"/>
+<pinref part="C3" gate="G$1" pin="2"/>
 </segment>
 <segment>
@@
 <wire x1="-93.98" y1="53.34" x2="-93.98" y2="50.8" width="0.1524" layer="91"/>
 <label x="-93.98" y="48.26" size="1.778" layer="95"/>
+</segment>
+<segment>
+<pinref part="C10" gate="G$1" pin="2"/>
+<wire x1="-182.88" y1="-7.62" x2="-182.88" y2="-10.16" width="0.1524" layer="91"/>
+<label x="-185.42" y="-12.7" size="1.778" layer="95"/>
 </segment>
 </net>
@@
 <net name="N$31" class="2">
 <segment>
-<pinref part="C7" gate="G$1" pin="1"/>
 <pinref part="R2" gate="G$1" pin="2"/>
 <wire x1="78.74" y1="55.88" x2="78.74" y2="60.96" width="0.1524" layer="91"/>
@@
 <wire x1="88.9" y1="60.96" x2="88.9" y2="55.88" width="0.1524" layer="91"/>
 <junction x="88.9" y="60.96"/>
+<pinref part="C3" gate="G$1" pin="1"/>
 </segment>
 </net>
@@
 <net name="N$33" class="2">
 <segment>
-<pinref part="C3" gate="G$1" pin="1"/>
 <pinref part="R7" gate="G$1" pin="2"/>
 <wire x1="-162.56" y1="55.88" x2="-162.56" y2="60.96" width="0.1524" layer="91"/>
@@
 <wire x1="-152.4" y1="60.96" x2="-152.4" y2="55.88" width="0.1524" layer="91"/>
 <junction x="-152.4" y="60.96"/>
+<pinref part="C17" gate="G$1" pin="1"/>
 </segment>
 </net>
 <net name="N$34" class="2">
 <segment>
-<pinref part="C5" gate="G$1" pin="1"/>
 <pinref part="R17" gate="G$1" pin="2"/>
 <wire x1="124.46" y1="-96.52" x2="124.46" y2="-91.44" width="0.1524" layer="91"/>
@@
 <wire x1="134.62" y1="-96.52" x2="134.62" y2="-91.44" width="0.1524" layer="91"/>
 <junction x="134.62" y="-91.44"/>
+<pinref part="C5" gate="G$1" pin="1"/>
 </segment>
 </net>
@@
 </segment>
 </net>
+<net name="TX0" class="0">
+<segment>
+<pinref part="U1" gate="G$1" pin="PE0(RXD0/PCINT8)"/>
+<wire x1="-83.82" y1="-20.32" x2="-91.44" y2="-20.32" width="0.1524" layer="91"/>
+<label x="-53.34" y="73.66" size="1.778" layer="95"/>
+<label x="-91.44" y="-20.32" size="1.778" layer="95"/>
+</segment>
+</net>

Commit message: fixed sch errors
Parts:
- removed C14, C15: 1uF, quadparts_prebuilt:CAPACITOR-NP_SMD-2012-0805_CERAMIC-1UF
- added C24, C9: 1uF, quadparts_prebuilt:CAPACITOR-NP_SMD-2012-0805_CERAMIC-1UF
- added C26, C27: 12pF, quadparts_prebuilt:CAPACITOR-NP_SMD-2012-0805_CERAMIC-12PF
- added R12: 10K, quadparts_prebuilt:RESISTOR_SMD-2012-0805-10K
Connections:
- new net N$36: R12.2, U2.SDA/SDI/SDO
- net 3V: now also C24.1, C9.1, R12.1
- net GND: now also C24.2, C26.2, C27.2, C9.2; no longer C14.2, C15.2
- net N$14: now also C26.1; no longer C14.1
- net N$5: now also C27.1; no longer C15.1
- net SDA: no longer U2.SDA/SDI/SDO
Changed lines of the file:
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@@
 <part name="GND10" library="quadparts_prebuilt" deviceset="GND" device=""/>
 <part name="Y1" library="quadparts_prebuilt" deviceset="CRYSTAL" device="5X3" value="16MHz"/>
-<part name="C14" library="quadparts_prebuilt" deviceset="CAPACITOR-NP_" device="SMD-2012-0805_CERAMIC-1UF" value="1uF"/>
-<part name="C15" library="quadparts_prebuilt" deviceset="CAPACITOR-NP_" device="SMD-2012-0805_CERAMIC-1UF" value="1uF"/>
 <part name="GND11" library="quadparts_prebuilt" deviceset="GND" device=""/>
 <part name="GND12" library="quadparts_prebuilt" deviceset="GND" device=""/>
@@
 <part name="C5" library="quadparts_prebuilt" deviceset="CAPACITOR-NP_" device="SMD-2012-0805_CERAMIC-0.1UF" value="0.1uF"/>
 <part name="C7" library="quadparts_prebuilt" deviceset="CAPACITOR-NP_" device="SMD-2012-0805_CERAMIC-0.1UF" value="0.1uF"/>
+<part name="C9" library="quadparts_prebuilt" deviceset="CAPACITOR-NP_" device="SMD-2012-0805_CERAMIC-1UF" value="1uF"/>
+<part name="C24" library="quadparts_prebuilt" deviceset="CAPACITOR-NP_" device="SMD-2012-0805_CERAMIC-1UF" value="1uF"/>
+<part name="GND27" library="quadparts_prebuilt" deviceset="GND" device=""/>
+<part name="GND28" library="quadparts_prebuilt" deviceset="GND" device=""/>
+<part name="R12" library="quadparts_prebuilt" deviceset="RESISTOR_" device="SMD-2012-0805-10K" value="10K"/>
+<part name="C26" library="quadparts_prebuilt" deviceset="CAPACITOR-NP_" device="SMD-2012-0805_CERAMIC-12PF" value="12pF"/>
+<part name="C27" library="quadparts_prebuilt" deviceset="CAPACITOR-NP_" device="SMD-2012-0805_CERAMIC-12PF" value="12pF"/>
 </parts>
 <sheets>
@@
 <instance part="GND10" gate="1" x="17.78" y="-35.56"/>
 <instance part="Y1" gate="G$1" x="-10.16" y="-22.86"/>
-<instance part="C14" gate="G$1" x="-15.24" y="-30.48"/>
-<instance part="C15" gate="G$1" x="-2.54" y="-30.48"/>
 <instance part="GND11" gate="1" x="-15.24" y="-40.64"/>
 <instance part="GND12" gate="1" x="-2.54" y="-40.64"/>
@@
 <instance part="C5" gate="G$1" x="124.46" y="-99.06"/>
 <instance part="C7" gate="G$1" x="-162.56" y="-99.06"/>
+<instance part="C9" gate="G$1" x="-63.5" y="40.64"/>
+<instance part="C24" gate="G$1" x="-53.34" y="40.64"/>
+<instance part="GND27" gate="1" x="-63.5" y="30.48"/>
+<instance part="GND28" gate="1" x="-53.34" y="30.48"/>
+<instance part="R12" gate="G$1" x="25.4" y="-111.76"/>
+<instance part="C26" gate="G$1" x="-15.24" y="-30.48"/>
+<instance part="C27" gate="G$1" x="-2.54" y="-30.48"/>
 </instances>
 <busses>
@@
 </segment>
 <segment>
-<pinref part="C14" gate="G$1" pin="2"/>
 <wire x1="-15.24" y1="-35.56" x2="-15.24" y2="-38.1" width="0.1524" layer="91"/>
 <pinref part="GND11" gate="1" pin="GND"/>
-</segment>
-<segment>
-<pinref part="C15" gate="G$1" pin="2"/>
+<pinref part="C26" gate="G$1" pin="2"/>
+</segment>
+<segment>
 <wire x1="-2.54" y1="-35.56" x2="-2.54" y2="-38.1" width="0.1524" layer="91"/>
 <pinref part="GND12" gate="1" pin="GND"/>
+<pinref part="C27" gate="G$1" pin="2"/>
 </segment>
 <segment>
@@
 <wire x1="38.1" y1="2.54" x2="38.1" y2="-7.62" width="0.1524" layer="91"/>
 </segment>
+<segment>
+<pinref part="GND27" gate="1" pin="GND"/>
+<pinref part="C9" gate="G$1" pin="2"/>
+<wire x1="-63.5" y1="33.02" x2="-63.5" y2="35.56" width="0.1524" layer="91"/>
+</segment>
+<segment>
+<pinref part="GND28" gate="1" pin="GND"/>
+<pinref part="C24" gate="G$1" pin="2"/>
+<wire x1="-53.34" y1="33.02" x2="-53.34" y2="35.56" width="0.1524" layer="91"/>
+</segment>
 </net>
 <net name="N$2" class="0">
@@
 <pinref part="U2" gate="G$1" pin="SDO_A/G"/>
 <wire x1="12.7" y1="-132.08" x2="12.7" y2="-116.84" width="0.1524" layer="91"/>
-<wire x1="12.7" y1="-116.84" x2="12.7" y2="-76.2" width="0.1524" layer="91"/>
+<wire x1="12.7" y1="-116.84" x2="12.7" y2="-111.76" width="0.1524" layer="91"/>
+<wire x1="12.7" y1="-111.76" x2="12.7" y2="-76.2" width="0.1524" layer="91"/>
 <wire x1="40.64" y1="-116.84" x2="12.7" y2="-116.84" width="0.1524" layer="91"/>
 <junction x="12.7" y="-116.84"/>
@@
 <wire x1="83.82" y1="-142.24" x2="58.42" y2="-142.24" width="0.1524" layer="91"/>
 <junction x="58.42" y="-142.24"/>
+<pinref part="R12" gate="G$1" pin="1"/>
+<wire x1="20.32" y1="-111.76" x2="12.7" y2="-111.76" width="0.1524" layer="91"/>
+<junction x="12.7" y="-111.76"/>
 </segment>
 <segment>
@@
 <label x="91.44" y="-7.62" size="1.778" layer="95"/>
 </segment>
+<segment>
+<pinref part="C9" gate="G$1" pin="1"/>
+<wire x1="-63.5" y1="43.18" x2="-63.5" y2="45.72" width="0.1524" layer="91"/>
+<label x="-63.5" y="45.72" size="1.778" layer="95" rot="R90" xref="yes"/>
+</segment>
+<segment>
+<pinref part="C24" gate="G$1" pin="1"/>
+<wire x1="-53.34" y1="43.18" x2="-53.34" y2="45.72" width="0.1524" layer="91"/>
+<label x="-53.34" y="45.72" size="1.778" layer="95" rot="R90" xref="yes"/>
+</segment>
 </net>
 <net name="N$10" class="0">
@@
 <wire x1="-7.62" y1="-22.86" x2="-2.54" y2="-22.86" width="0.1524" layer="91"/>
 <junction x="-2.54" y="-22.86"/>
-<pinref part="C15" gate="G$1" pin="1"/>
+<pinref part="C27" gate="G$1" pin="1"/>
 </segment>
 </net>
@@
 <wire x1="-27.94" y1="-17.78" x2="-15.24" y2="-17.78" width="0.1524" layer="91"/>
 <wire x1="-15.24" y1="-17.78" x2="-15.24" y2="-22.86" width="0.1524" layer="91"/>
-<pinref part="C14" gate="G$1" pin="1"/>
+<pinref part="C26" gate="G$1" pin="1"/>
 </segment>
 </net>
@@
 <wire x1="-83.82" y1="0" x2="-91.44" y2="0" width="0.1524" layer="91"/>
 <label x="-91.44" y="0" size="1.778" layer="95"/>
-</segment>
-<segment>
-<pinref part="U2" gate="G$1" pin="SDA/SDI/SDO"/>
-<wire x1="40.64" y1="-111.76" x2="22.86" y2="-111.76" width="0.1524" layer="91"/>
-<label x="22.86" y="-111.76" size="1.778" layer="95"/>
 </segment>
 </net>
@@
 </segment>
 </net>
+<net name="N$36" class="0">
+<segment>
+<pinref part="U2" gate="G$1" pin="SDA/SDI/SDO"/>
+<pinref part="R12" gate="G$1" pin="2"/>
+<wire x1="40.64" y1="-111.76" x2="30.48" y2="-111.76" width="0.1524" layer="91"/>
+</segment>
+</net>

Commit message: Fixed board errors
Connections:
- net BAT_GND: now also D5.C, D6.C; no longer D10.C, D9.C
- net GND: now also D10.C, D9.C; no longer D5.C, D6.C
- net N$18: now also D9.A, R9.2; no longer D10.A, R10.2
- net N$19: now also D10.A, R5.1; no longer D5.A, R9.2
- net N$27: now also D5.A, R10.2; no longer D9.A, R11.1
- net N$28: now also R11.1; no longer R5.1
Other:
- moved on the sheet: D10, D5, D6, D9
Changed lines of the file:
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@@
 <instance part="GND23" gate="1" x="99.06" y="-127"/>
 <instance part="J3" gate="G$1" x="78.74" y="-25.4"/>
-<instance part="D9" gate="G$1" x="-109.22" y="60.96" rot="R270"/>
-<instance part="D10" gate="G$1" x="-93.98" y="60.96" rot="R270"/>
-<instance part="D5" gate="G$1" x="-106.68" y="-71.12" rot="R270"/>
-<instance part="D6" gate="G$1" x="-109.22" y="-20.32" rot="R90"/>
+<instance part="D9" gate="G$1" x="-106.68" y="-71.12" rot="R270"/>
+<instance part="D10" gate="G$1" x="-109.22" y="-17.78" rot="R90"/>
+<instance part="D5" gate="G$1" x="-93.98" y="63.5" rot="R270"/>
+<instance part="D6" gate="G$1" x="-109.22" y="66.04" rot="R270"/>
 <instance part="GND24" gate="1" x="-106.68" y="-83.82"/>
 <instance part="GND25" gate="1" x="-116.84" y="-7.62"/>
@@
 </segment>
 <segment>
-<pinref part="D5" gate="G$1" pin="C"/>
-<wire x1="-106.68" y1="-78.74" x2="-106.68" y2="-81.28" width="0.1524" layer="91"/>
-<pinref part="GND24" gate="1" pin="GND"/>
-</segment>
-<segment>
 <pinref part="GND21" gate="1" pin="GND"/>
 <pinref part="C23" gate="G$1" pin="2"/>
@@
 <segment>
 <pinref part="GND25" gate="1" pin="GND"/>
-<pinref part="D6" gate="G$1" pin="C"/>
 <wire x1="-116.84" y1="-5.08" x2="-109.22" y2="-5.08" width="0.1524" layer="91"/>
-<wire x1="-109.22" y1="-5.08" x2="-109.22" y2="-12.7" width="0.1524" layer="91"/>
+<pinref part="D10" gate="G$1" pin="C"/>
+<wire x1="-109.22" y1="-5.08" x2="-109.22" y2="-10.16" width="0.1524" layer="91"/>
 </segment>
 <segment>
@@
 <pinref part="C24" gate="G$1" pin="2"/>
 <wire x1="-53.34" y1="33.02" x2="-53.34" y2="35.56" width="0.1524" layer="91"/>
+</segment>
+<segment>
+<pinref part="D9" gate="G$1" pin="C"/>
+<pinref part="GND24" gate="1" pin="GND"/>
+<wire x1="-106.68" y1="-78.74" x2="-106.68" y2="-81.28" width="0.1524" layer="91"/>
 </segment>
 </net>
@@
 </segment>
 <segment>
-<pinref part="D9" gate="G$1" pin="C"/>
-<wire x1="-109.22" y1="53.34" x2="-109.22" y2="50.8" width="0.1524" layer="91"/>
-<label x="-109.22" y="48.26" size="1.778" layer="95"/>
-</segment>
-<segment>
-<pinref part="D10" gate="G$1" pin="C"/>
-<wire x1="-93.98" y1="53.34" x2="-93.98" y2="50.8" width="0.1524" layer="91"/>
-<label x="-93.98" y="48.26" size="1.778" layer="95"/>
-</segment>
-<segment>
 <pinref part="C10" gate="G$1" pin="2"/>
 <wire x1="-182.88" y1="-7.62" x2="-182.88" y2="-10.16" width="0.1524" layer="91"/>
 <label x="-185.42" y="-12.7" size="1.778" layer="95"/>
+</segment>
+<segment>
+<pinref part="D6" gate="G$1" pin="C"/>
+<wire x1="-109.22" y1="58.42" x2="-109.22" y2="55.88" width="0.1524" layer="91"/>
+<label x="-109.22" y="55.88" size="1.778" layer="95" rot="R270" xref="yes"/>
+</segment>
+<segment>
+<pinref part="D5" gate="G$1" pin="C"/>
+<wire x1="-93.98" y1="55.88" x2="-93.98" y2="53.34" width="0.1524" layer="91"/>
+<label x="-93.98" y="53.34" size="1.778" layer="95" rot="R270" xref="yes"/>
 </segment>
 </net>
@@
 </segment>
 </net>
-<net name="N$27" class="0">
-<segment>
-<pinref part="D9" gate="G$1" pin="A"/>
-<wire x1="-109.22" y1="78.74" x2="-109.22" y2="68.58" width="0.1524" layer="91"/>
-<pinref part="R11" gate="G$1" pin="1"/>
-</segment>
-</net>
-<net name="N$19" class="0">
-<segment>
-<wire x1="-106.68" y1="-60.96" x2="-106.68" y2="-63.5" width="0.1524" layer="91"/>
-<pinref part="D5" gate="G$1" pin="A"/>
-<pinref part="R9" gate="G$1" pin="2"/>
-</segment>
-</net>
-<net name="N$28" class="0">
-<segment>
-<wire x1="-109.22" y1="-30.48" x2="-109.22" y2="-27.94" width="0.1524" layer="91"/>
-<pinref part="D6" gate="G$1" pin="A"/>
-<pinref part="R5" gate="G$1" pin="1"/>
-</segment>
-</net>
-<net name="N$18" class="0">
-<segment>
-<pinref part="D10" gate="G$1" pin="A"/>
-<wire x1="-93.98" y1="73.66" x2="-93.98" y2="68.58" width="0.1524" layer="91"/>
-<pinref part="R10" gate="G$1" pin="2"/>
-</segment>
-</net>
 <net name="N$23" class="0">
 <segment>
@@
 </segment>
 </net>
+<net name="N$18" class="0">
+<segment>
+<pinref part="R9" gate="G$1" pin="2"/>
+<pinref part="D9" gate="G$1" pin="A"/>
+<wire x1="-106.68" y1="-60.96" x2="-106.68" y2="-63.5" width="0.1524" layer="91"/>
+</segment>
+</net>
+<net name="N$19" class="0">
+<segment>
+<pinref part="D10" gate="G$1" pin="A"/>
+<pinref part="R5" gate="G$1" pin="1"/>
+<wire x1="-109.22" y1="-25.4" x2="-109.22" y2="-30.48" width="0.1524" layer="91"/>
+</segment>
+</net>
+<net name="N$27" class="0">
+<segment>
+<pinref part="R10" gate="G$1" pin="2"/>
+<pinref part="D5" gate="G$1" pin="A"/>
+<wire x1="-93.98" y1="73.66" x2="-93.98" y2="71.12" width="0.1524" layer="91"/>
+</segment>
+</net>
+<net name="N$28" class="0">
+<segment>
+<pinref part="R11" gate="G$1" pin="1"/>
+<pinref part="D6" gate="G$1" pin="A"/>
+<wire x1="-109.22" y1="78.74" x2="-109.22" y2="73.66" width="0.1524" layer="91"/>
+</segment>
+</net>
